File: cad_files/wiring/wiring.sch (KiCad schematic (older format))
At the start: 64 parts, among them K1 Finder 40.51.9.012.0000, K1a1 auxcontalt, K2 Finder 40.51.9.012.0000, K2a1 auxcontalt, K3 Finder 40.51.9.012.0000, K3a1 auxcontalt, K4 Finder 40.51.9.012.0000, K4a1 auxcontalt, P1 screw_conn, P10 screw_conn, P101 CONN_01X05, P102 CONN_01X02, P103 CONN_01X02, P104 CONN_01X02, P105 CONN_01X03, P106 CONN_01X02, P107 CONN_01X02, P108 CONN_01X02, P109 CONN_01X05, P11 screw_conn, P12 screw_conn, P13 screw_conn, P14 screw_conn, P15 screw_conn, P16 screw_conn, P17 screw_conn, P18 DB9, P2 screw_conn, P201 CONN_01X02, P202 CONN_01X01, P203 CONN_01X01, P204 CONN_01X06, P205 CONN_01X03, P206 CONN_01X03, P207 CONN_01X03, P208 CONN_01X01, P209 CONN_01X01, P3 screw_conn, P4 screw_conn, P5 screw_conn, P6 screw_conn, P7 screw_conn, P8 screw_conn, P9 screw_conn, SW1 auxcontalt, SW2 auxcontalt, SW3 auxcontalt, SW4 auxcontalt

Commit message: 231023
Parts:
- added R1: *, symbol Device:R
- AK1, AK2, AK3, K1a1, K2a1, K3a1, K4a1: symbol auxcontalt -> pzs_others:auxcontalt
- BT1: symbol Battery -> wiring-rescue:Battery
- F1, F2, F3: symbol overcurrent_breaker -> pzs_others:overcurrent_breaker
- F4, F5, F6: symbol Fuse -> wiring-rescue:Fuse
- K1, K2, K3, K4: symbol electromagnetic_actor_1 -> pzs_others:electromagnetic_actor_1
- LS1: symbol Speaker_Ultrasound -> wiring-rescue:Speaker_Ultrasound
- P1, P10, P11, P12, P13, P14, P15, P16, P17, P2, P3, P4, P5, P6, P7, P8, P9: symbol screw_conn -> pzs_others:screw_conn
- P101, P109: symbol CONN_01X05 -> Connector:Conn_01x05_Female
- P102, P103, P104, P106, P107, P108, P201: symbol CONN_01X02 -> Connector:Conn_01x02_Female
- P105, P205, P206, P207: symbol CONN_01X03 -> Connector:Conn_01x03_Female
- P18: symbol DB9 -> wiring-rescue:DB9
- P202, P203, P208, P209: symbol CONN_01X01 -> Connector:Conn_01x01_Female
- P204: symbol CONN_01X06 -> Connector:Conn_01x06_Female
- SW1, SW2, SW3: symbol auxcontalt -> Switch:SW_DPDT_x2
- SW1: renamed from SW'1; symbol auxcontalt -> Switch:SW_DPDT_x2
- SW2: renamed from SW'2; symbol auxcontalt -> Switch:SW_DPDT_x2
- SW3: renamed from SW'3; symbol auxcontalt -> Switch:SW_DPDT_x2
- SW4: symbol auxcontalt -> Switch:SW_SP3T
- Tr1, Tr2: symbol transformer_1P_1S -> pzs_others:transformer_1P_1S
Connections:
- net at P13.1: now also P101.2 (Pin_2); no longer P101.5 (P5)
- net at P204.2 (Pin_2): now also SW1.3 (C); no longer SW1.~ (B)
- net at P101.3 (Pin_3): now also SW1.4 (A); no longer SW1.~ (B)
- net at P204.4 (Pin_4): now also SW2.3 (C); no longer SW2.~ (B)
- net at P204.6 (Pin_6): now also SW3.3 (C); no longer SW3.~ (B)
- new net: AK1.~ (B), AK2.~ (B), AK3.~ (B), P208.1 (Pin_1)
- new net: F4.1, Tr1.~, Tr2.~
- new net: P207.1 (Pin_1), SW1.2 (B), SW2.2 (B), SW3.2 (B)
- new net: SW1.5 (B), SW2.4 (A)
- new net: P209.1 (Pin_1), SW1.6 (C), SW2.6 (C), SW3.6 (C)
- new net: SW2.5 (B), SW3.4 (A)
- new net: P206.2 (Pin_2), R1.2, SW3.5 (B), SW4.4
- new net: R1.1, SW4.1
- new net: P101.5 (Pin_5), SW4.3
Other:
- note added: "Manual operation"
- note added: "Sign lights"
- note removed: "Manual operation mode"
- note removed: "Status lamp"
- moved on the sheet: P202, P203, P208, P209
